File: pebble_qi_eagle/pebble_qi_eagle.brd (EAGLE design)
At the start: 160 x 100 mm, 17 parts

Commit message: Initial routing
Routing:
- net N$12: track 0.00 -> 63.5 mm
- net GND: track 0.00 -> 47.1 mm
- net N$1: track 0.00 -> 20.8 mm
- net N$2: track 0.00 -> 20.7 mm
- net N$7: track 0.00 -> 18.0 mm
- net N$13: track 0.00 -> 17.8 mm
- net N$16: track 0.00 -> 9.19 mm
- net N$11: track 0.00 -> 6.13 mm
- net N$5: track 0.00 -> 5.46 mm
- net N$10: track 0.00 -> 4.86 mm
- net N$3: track 0.00 -> 4.43 mm
- net N$6: track 0.00 -> 4.29 mm
- net N$4: track 0.00 -> 3.87 mm
- net N$9: track 0.00 -> 3.30 mm
